File: 68030-design/kicad/duart_spi_rtc.kicad_sch (KiCad schematic)
At the start: 22 parts, among them J7 TTL-232, J8 TTL-232, J9 SPI NIC, U22 SN74LVC125ADR, U23 DS3234S#, U6 SC26C92A1A

Commit message: PCB: condense to 220x175 mm with SMD oscillators, IDE buffers, battery holder, fuse
Parts:
- BT1: footprint Battery:BatteryHolder_Keystone_103_1x20mm -> Battery:BatteryHolder_Keystone_3034_1x20mm; MPN Keystone 103 -> Keystone 3034
Changed lines of the file:
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@@
 			)
 		)
-		(property "Footprint" "Battery:BatteryHolder_Keystone_103_1x20mm"
+		(property "Footprint" "Battery:BatteryHolder_Keystone_3034_1x20mm"
 			(at 309.88 193.04 0)
 			(effects
@@
 			)
 		)
-		(property "MPN" "Keystone 103"
+		(property "MPN" "Keystone 3034"
 			(at 309.88 193.04 0)
 			(effects
