File: 68030-design/kicad/ide.kicad_sch (KiCad schematic)
At the start: 22 parts, among them J6 IDE 40-pin, U11 SN74ACT245N, U12 SN74ACT245N, U13 SN74ACT245N

Commit message: PCB: condense to 220x175 mm with SMD oscillators, IDE buffers, battery holder, fuse
Parts:
- U11, U12, U13: value SN74ACT245N -> SN74ACT245DW; footprint Package_DIP:DIP-20_W7.62mm -> Package_SO:SOIC-20W_7.5x12.8mm_P1.27mm; MPN SN74ACT245N -> SN74ACT245DW; Note TI SCAS452H, PDIP (N), active. Same 245 pinout; footprint s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 -> TI SCAS452H SOIC (DW). Same 245 pinout as the N part. Reel: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
Changed lines of the file:
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@@
 			)
 		)
-		(property "Value" "SN74ACT245N"
+		(property "Value" "SN74ACT245DW"
 			(at 70 119 0)
 			(effects
@@
 			)
 		)
-		(property "Footprint" "Package_DIP:DIP-20_W7.62mm"
+		(property "Footprint" "Package_SO:SOIC-20W_7.5x12.8mm_P1.27mm"
 			(at 90.17 95.25 0)
 			(effects
@@
 			)
 		)
-		(property "MPN" "SN74ACT245N"
+		(property "MPN" "SN74ACT245DW"
 			(at 90.17 95.25 0)
 			(effects
@@
 			)
 		)
-		(property "Note" "TI SCAS452H, PDIP (N), active. Same 245 pinout; footprint stays DIP-20. Fig. 6-1 CL=50 pF only"
+		(property "Note" "TI SCAS452H SOIC (DW). Same 245 pinout as the N part. Reel: SN74ACT245DWR [VERIFY stock]"
 			(at 90.17 95.25 0)
 			(effects
@@
 			)
 		)
-		(property "Value" "SN74ACT245N"
+		(property "Value" "SN74ACT245DW"
 			(at 70 209 0)
 			(effects
@@
 			)
 		)
-		(property "Footprint" "Package_DIP:DIP-20_W7.62mm"
+		(property "Footprint" "Package_SO:SOIC-20W_7.5x12.8mm_P1.27mm"
 			(at 90.17 185.42 0)
 			(effects
@@
 			)
 		)
-		(property "MPN" "SN74ACT245N"
+		(property "MPN" "SN74ACT245DW"
 			(at 90.17 185.42 0)
 			(effects
@@
 			)
 		)
-		(property "Note" "TI SCAS452H, PDIP (N), active. Same 245 pinout; footprint stays DIP-20. Fig. 6-1 CL=50 pF only"
+		(property "Note" "TI SCAS452H SOIC (DW). Same 245 pinout as the N part. Reel: SN74ACT245DWR [VERIFY stock]"
 			(at 90.17 185.42 0)
 			(effects
@@
 			)
 		)
-		(property "Value" "SN74ACT245N"
+		(property "Value" "SN74ACT245DW"
 			(at 70 304 0)
 			(effects
@@
 			)
 		)
-		(property "Footprint" "Package_DIP:DIP-20_W7.62mm"
+		(property "Footprint" "Package_SO:SOIC-20W_7.5x12.8mm_P1.27mm"
 			(at 90.17 279.4 0)
 			(effects
@@
 			)
 		)
-		(property "MPN" "SN74ACT245N"
+		(property "MPN" "SN74ACT245DW"
 			(at 90.17 279.4 0)
 			(effects
@@
 			)
 		)
-		(property "Note" "TI SCAS452H, PDIP (N), active. Same 245 pinout; footprint stays DIP-20. Fig. 6-1 CL=50 pF only"
+		(property "Note" "TI SCAS452H SOIC (DW). Same 245 pinout as the N part. Reel: SN74ACT245DWR [VERIFY stock]"
 			(at 90.17 279.4 0)
 			(effects
