File: 68030-design/kicad/m68030-sbc.kicad_pcb (KiCad board)
At the start: 4 copper layers, 275 x 215 mm, 292 parts, among them J1 SIMM-72 socket, J10 DIN41612-C-96, J11 LA1 A31-A0, J12 LA2 D31-D0, J13 LA3 control, J2 9-24V DC, J3 5V_BENCH, J4 JTAG (ATDH1150USB), J5 JTAG U4 (ATDH1150USB), J6 IDE 40-pin, J7 TTL-232, J8 TTL-232, J9 SPI NIC, Q1 SUD50P04-08, SW1 WARM_RESET, SW2 NMI, SW3 COLD_RESET, U1 MC68030RC33C, U10 74ACT244, U11 SN74ACT245N, U12 SN74ACT245N, U13 SN74ACT245N, U14 SN74ACT244DW, U15 SN74ACT244DW, U16 SN74ACT244DW, U17 SN74ACT244DW, U18 SN74ACT245DW, U19 SN74ACT245DW, U2 MC68882FN33A, U20 SN74ACT245DW, U21 SN74ACT245DW, U22 SN74LVC125ADR, U23 DS3234S#, U27 TPS3808G50DBVR, U3 ATF1508AS-7JX84, U4 ATF1508AS-7JX84, U5 SST39SF040-70-4C-NHE, U6 SC26C92A1A, U7 TPS3702CX50DDCR, U8 LM2678S-5.0, U801 74ACT257, U802 74ACT257, U803 74ACT257, U9 AMS1117-3.3, X1 25.000MHz, X2 50.000MHz, X3 FPU osc (DNP), Y1 3.6864MHz

Commit message: PCB: add silkscreen labels for connectors and jumpers
Other:
- board text added: "+"
- board text added: "+5V"
- board text added: "3V3"
- board text added: "5V"
- board text added: "5V BENCH IN"
- board text added: "BUCK OFF"
- board text added: "CBACK"
- board text added: "CDIS"
- board text added: "CPU"
- board text added: "CS"
- board text added: "CTS"
- board text added: "DS"
- board text added: "EXPANSION DIN-41612"
- board text added: "FPU CLK"
- board text added: "GND"
- board text added: "IDE 40-PIN"
- board text added: "INT"
- board text added: "ISO"
- board text added: "JP801 STERM JP802 CBREQ"
- board text added: "JTAG DRAM U4"
- board text added: "JTAG GLUE U3"
- board text added: "LA1 A31-A0"
- board text added: "LA2 D31-D0"
- board text added: "LA3 CTRL"
- board text added: "MISO"
- board text added: "MMUDIS"
- board text added: "MOSI"
- board text added: "NC"
- board text added: "PWR IN 9-24V DC"
- board text added: "RST"
- board text added: "RST SET"
- board text added: "RTS"
- board text added: "RXD"
- board text added: "SCK"
- board text added: "SERIAL A TTL"
- board text added: "SERIAL B TTL"
- board text added: "SIMM 72 DRAM"
- board text added: "SPI NIC"
- board text added: "TXD"
- board text added: "X3"

Commit message: PCB: condense to 220x175 mm with SMD oscillators, IDE buffers, battery holder, fuse
Parts:
- BT1: footprint Battery:BatteryHolder_Keystone_103_1x20mm -> Battery:BatteryHolder_Keystone_3034_1x20mm
- F1: value T5A 5x20 -> T5A 0454005.MR; footprint Fuse:Fuseholder_Cylinder-5x20mm_Schurter_0031_8201_Horizontal_Open -> Fuse:Fuse_Littelfuse-NANO2-451_453
- U11, U12, U13: value SN74ACT245N -> SN74ACT245DW; footprint Package_DIP:DIP-20_W7.62mm -> Package_SO:SOIC-20W_7.5x12.8mm_P1.27mm
- X1, X2, X3: footprint Oscillator:Oscillator_DIP-14 -> m68030-sbc:Oscillator_SMD_ECS-3951M_7.0x5.0mm_DIP14PinMap
- moved U7 173.3 mm to (172.1, 7.41)
- moved C810 172.8 mm to (64.4, 16.4), turned to 0 degrees
- moved U27 157.7 mm to (171.4, 12.0)
- moved C402 156.8 mm to (181.9, 18.6)
- moved BT1 152.6 mm to (88.0, 150.0)
- moved R402 151.5 mm to (176.7, 23.4)
- moved JP401 149.5 mm to (174.9, 18.1)
- moved C401 147.8 mm to (168.9, 18.7), turned to 90 degrees
- moved C819 133.9 mm to (88.7, 35.8), turned to 0 degrees
- moved C813 129.6 mm to (89.8, 41.2), turned to 90 degrees
- moved JP3 126.4 mm to (134.5, 45.0), turned to 90 degrees
- moved X2 115.7 mm to (139.0, 56.0)
- moved C304 113.6 mm to (134.9, 60.7), turned to 0 degrees
- moved C517 113.1 mm to (78.7, 51.6)
- moved C303 112.3 mm to (133.5, 53.1)
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Routing:
- net GND: track 201.3 -> 212.7 mm, vias 151 -> 175
- net +5V: track 231.9 -> 230.3 mm, vias 138 -> 148
Other:
- board size 275 x 215 mm -> 220 x 175 mm
- board text added: "BUCK ISO"
- board text added: "DNP: X3, U801-U803, J3. JP801-804 / JP701-703 open."
- board text added: "HEATSINK 40x40 mm on U1. Top-side keepout."
- board text added: "SIMM locating holes UNVERIFIED (NPTH as drawn). J10 VERIFY vs HARTING 09032966821."
- board text added: "STERM"
- board text added: "m68030-sbc Rev A 4-layer 220 x 175 mm"
- board text removed: "DNP: X3, U801 U802 U803 (74ACT257 mux fallback). JP801-804 and JP701-703 open."
- board text removed: "HEATSINK stick-on 40x40 mm centered on U1. Keep other top-side parts outside this outline. PGA thetaJA ~30 C/W, up to 2.6 W (spec 6.3)."
- board text removed: "ISO"
- board text removed: "J10 footprint is KiCad DIN41612_C_3x32_Female_Vertical_THT. VERIFY against HARTING 09032966821 before ordering."
- board text removed: "SIMM locating holes UNVERIFIED: NPTH as drawn (1.63 / 2.41 mm). Do not treat as plated. Print 1:1 vs TE 5822021 / 114-1061."
- board text removed: "m68030-sbc Rev A 4-layer 275 x 215 mm"
