File: 68030-design/kicad/power.kicad_sch (KiCad schematic)
At the start: 29 parts, among them J2 9-24V DC, J3 5V_BENCH, Q1 SUD50P04-08, U8 LM2678S-5.0, U9 AMS1117-3.3

Commit message: PCB: condense to 220x175 mm with SMD oscillators, IDE buffers, battery holder, fuse
Parts:
- F1: value T5A 5x20 -> T5A 0454005.MR; footprint Fuse:Fuseholder_Cylinder-5x20mm_Schurter_0031_8201_Horizontal_Open -> Fuse:Fuse_Littelfuse-NANO2-451_453; MPN 5x20 mm time-lag 5 A glass fuse + Schurter 0031.8201 holder -> Littelfuse 0454005.MR
Changed lines of the file:
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@@
 			)
 		)
-		(property "Value" "T5A 5x20"
+		(property "Value" "T5A 0454005.MR"
 			(at 53.34 78.74 90)
 			(effects
@@
 			)
 		)
-		(property "Footprint" "Fuse:Fuseholder_Cylinder-5x20mm_Schurter_0031_8201_Horizontal_Open"
+		(property "Footprint" "Fuse:Fuse_Littelfuse-NANO2-451_453"
 			(at 53.34 76.2 0)
 			(effects
@@
 			)
 		)
-		(property "MPN" "5x20 mm time-lag 5 A glass fuse + Schurter 0031.8201 holder"
+		(property "MPN" "Littelfuse 0454005.MR"
 			(at 53.34 76.2 0)
 			(effects
