File: 68030-design/kicad/glue_cpld.kicad_sch (KiCad schematic)
At the start: 28 parts, among them J4 JTAG (ATDH1150USB), U3 ATF1508AS-7JX84

Commit message: CPLD: Rev A.2 pin swap for U3 glue and U4 DRAM to match the 220x175 placement
Re-assign the U3/U4 user I/O pins to follow the bus order at the CPU, FPU,
SIMM, LA headers and DIN. Dedicated inputs, JTAG, power, jumpered pins, TP pins
and the reserved SPI pins (46/48/49) did not move.

- U3 glue: 57 pins moved; airwire length 2784 -> 2369 mm, crossings 254 -> 0.
- U4 DRAM: 54 pins moved; 1598 -> 1296 mm, crossings 372 -> 8. The search
  kept fit1508 in the loop, so all 9 cascades and the 14.0 ns timing were kept.
- Refits (fit1508 v1918, -7, JTAG on): glue 121/128 MC, 20.3 ns; DRAM 78/128 MC,
  14.0 ns (same as Rev A.1). All CPLD and system sims: 0 errors, 0 DSACK contention.
- Schematics: label edits in place in glue_cpld/dram.kicad_sch (not build.py).
  ERC 0 errors / 0 warnings.
- PCB: 111 U3/U4 pad nets updated; R804-R824 moved to B.Cu in SIMM pin order.
  DRC 0 errors, parity 0 (board still unrouted at this commit).
- FreeRouting re-test (scratch): 4L completion 27 % -> 32.5 %, 6L 25 % -> 29.9 %.
- New tools: kicad/tools/cpld_pinswap_*.py. Pin tables in cpld/*/README.md.
- .kicad_pro unchanged.
Connections:
- net A1: now also U3.80 (I/O); no longer U3.31 (I/O)
- net A13: now also U3.31 (I/O); no longer U3.28 (I/O)
- net A14: now also U3.36 (I/O); no longer U3.27 (I/O)
- net A15: now also U3.24 (I/O); no longer U3.25 (I/O)
- net A16: now also U3.22 (I/O); no longer U3.24 (I/O)
- net A17: now also U3.35 (I/O); no longer U3.22 (I/O)
- net A18: now also U3.33 (I/O); no longer U3.21 (I/O)
- net A19: now also U3.17 (I/O); no longer U3.20 (I/O)
- net A2: now also U3.28 (I/O); no longer U3.30 (I/O)
- net A27: now also U3.79 (I/O); no longer U3.18 (I/O)
- net A28: now also U3.75 (I/O); no longer U3.17 (I/O)
- net A29: now also U3.74 (I/O); no longer U3.16 (I/O)
- net A3: now also U3.30 (I/O); no longer U3.29 (I/O)
- net A30: now also U3.77 (I/O); no longer U3.15 (I/O)
- net A31: now also U3.76 (I/O); no longer U3.12 (I/O/PD1)
- net AVEC_n: now also U3.6 (I/O); no longer U3.75 (I/O)
- net BERR_n: now also U3.65 (I/O); no longer U3.11 (I/O)
- net BUS_RD_n: now also U3.34 (I/O); no longer U3.58 (I/O)
- net BUS_WR_n: now also U3.39 (I/O); no longer U3.60 (I/O)
- net CIIN_n: now also U3.61 (I/O); no longer U3.76 (I/O)
- net DRAM_SEL_n: now also U3.5 (I/O); no longer U3.55 (I/O)
- net DSACK0_n: now also U3.8 (I/O); no longer U3.9 (I/O)
- net DSACK1_n: now also U3.81 (I/O/GCLK3); no longer U3.10 (I/O)
- net DUART_CS_n: now also U3.51 (I/O); no longer U3.61 (I/O)
- net DUART_INT_n: now also U3.37 (I/O); no longer U3.33 (I/O)
- net DUART_RST: now also U3.45 (I/O/PD2); no longer U3.39 (I/O)
- net EXP_BUF_EN_n: now also U3.20 (I/O); no longer U3.70 (I/O)
- net EXP_INT_n: now also U3.16 (I/O); no longer U3.35 (I/O)
- net EXP_SEL_n: now also U3.12 (I/O/PD1); no longer U3.69 (I/O)
- net FC0: now also U3.11 (I/O); no longer U3.6 (I/O)
- net FC1: now also U3.10 (I/O); no longer U3.5 (I/O)
- net FC2: now also U3.9 (I/O); no longer U3.4 (I/O)
- net FPU_CS_n: now also U3.67 (I/O); no longer U3.56 (I/O)
- net HALT_LED_n: now also U3.44 (I/O); no longer U3.45 (I/O/PD2)
- net HALT_n: now also U3.64 (I/O); no longer U3.54 (I/O)
- net IDE_BUF_EN_n: now also U3.50 (I/O); no longer U3.68 (I/O)
- net IDE_CS0_n: now also U3.55 (I/O); no longer U3.63 (I/O)
- net IDE_CS1_n: now also U3.52 (I/O); no longer U3.64 (I/O)
- net IDE_DA0: now also U3.63 (I/O); no longer U3.50 (I/O)
- net IDE_DA1: now also U3.60 (I/O); no longer U3.51 (I/O)
- net IDE_DA2: now also U3.57 (I/O); no longer U3.52 (I/O)
- net IDE_DIOR_n: now also U3.21 (I/O); no longer U3.65 (I/O)
- net IDE_DIOW_n: now also U3.58 (I/O); no longer U3.67 (I/O)
- net IDE_INTRQ: now also U3.54 (I/O); no longer U3.73 (I/O)
- net IDE_IORDY: now also U3.56 (I/O); no longer U3.74 (I/O)
- net IPL0_n: now also U3.68 (I/O); no longer U3.77 (I/O)
- net IPL1_n: now also U3.4 (I/O); no longer U3.79 (I/O)
- net IPL2_n: now also U3.70 (I/O); no longer U3.80 (I/O)
- net LED_n: now also U3.29 (I/O); no longer U3.40 (I/O)
- net NIC_INT_n: now also U3.41 (I/O); no longer U3.34 (I/O)
- net NMI_BTN_n: now also U3.25 (I/O); no longer U3.36 (I/O)
- net PERIPH_RST_n: now also U3.15 (I/O); no longer U3.37 (I/O)
- net RESET_n: now also U3.73 (I/O); no longer U3.81 (I/O/GCLK3)
- net ROM_CE_n: now also U3.40 (I/O); no longer U3.57 (I/O)
- net R_W: now also U3.18 (I/O); no longer U3.8 (I/O)
- net STATUS_n: now also U3.69 (I/O); no longer U3.44 (I/O)
- net WARM_RST_BTN_n: now also U3.27 (I/O); no longer U3.41 (I/O)
Other:
- note added: "FITTED PINOUT: Yosys 0.52 + hoglet67/atf15xx_yosys -> Microchip fit1508.exe v1918 (Wine 10), ATF1508AS PLCC84 -7, JTAG ON, pins locked (-preassign keep), -pin_keep on, -optimize off. Rev A.1 (2026-09-27): 121/128 macrocells, 62 flip-flops, 322 product terms; 57/60 user I/O + 4 JTAG + 4/4 dedicated inputs. Rev A.2 (2026-10-17): same logic, I/O pins re-assigned for the 220x175 layout; still 121/128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"
- note added: "Rev A.2 pin swap (2026-10-17): I/O pins re-assigned to the 220x175 placement (cpld/glue/pinout.md). IDE_DA0/1/2 (registered IDE address -> ide sheet U13) are now pins 63/60/57. Pins 46/48/49: reserved CPLD SPI master (spec 1.4), behind open solder jumpers."
- note removed: "FITTED PINOUT: Yosys 0.52 + hoglet67/atf15xx_yosys -> Microchip fit1508.exe v1918 (Wine 10), ATF1508AS PLCC84 -7, JTAG ON, pins locked (-preassign keep), -pin_keep on, -optimize off. Rev A.1 (2026-09-27): 121/128 macrocells, 62 flip-flops, 322 product terms; 57/60 user I/O + 4 JTAG + 4/4 dedicated inputs. Sources, reports, JEDEC: cpld/glue/ (glue.v, glue.fit, glue.jed, pinout.csv). No series resi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"
- note removed: "Pins 50-52: IDE_DA0-2, registered IDE address (Rev A.1, was spare/TP707-709) -> ide sheet (U13). Pins 46/48/49: reserved CPLD SPI master (spec 1.4), behind open solder jumpers."
