File: 68030-design/kicad/clock.kicad_sch (KiCad schematic)
At the start: 22 parts, among them U10 74ACT244, X1 25.000MHz, X2 50.000MHz, X3 FPU osc (DNP), Y1 3.6864MHz

Commit message: PCB: condense to 220x175 mm with SMD oscillators, IDE buffers, battery holder, fuse
Parts:
- X1: footprint Oscillator:Oscillator_DIP-14 -> m68030-sbc:Oscillator_SMD_ECS-3951M_7.0x5.0mm_DIP14PinMap; MPN 25.000 MHz 5 V CMOS full-can oscillator (socketed) -> ECS-3951M-250-BN-TR
- X2: footprint Oscillator:Oscillator_DIP-14 -> m68030-sbc:Oscillator_SMD_ECS-3951M_7.0x5.0mm_DIP14PinMap; MPN 50.000 MHz 5 V CMOS oscillator -> ECS-3951M-500-BN-TR
- X3: footprint Oscillator:Oscillator_DIP-14 -> m68030-sbc:Oscillator_SMD_ECS-3951M_7.0x5.0mm_DIP14PinMap; MPN optional 5 V CMOS oscillator for a slower 68882 -> ECS-3951M-200-BN-TR [VERIFY freq vs 68882 grade]
Changed lines of the file:
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@@
 			)
 		)
-		(property "Footprint" "Oscillator:Oscillator_DIP-14"
+		(property "Footprint" "m68030-sbc:Oscillator_SMD_ECS-3951M_7.0x5.0mm_DIP14PinMap"
 			(at 68.58 76.2 0)
 			(effects
@@
 			)
 		)
-		(property "MPN" "25.000 MHz 5 V CMOS full-can oscillator (socketed)"
+		(property "MPN" "ECS-3951M-250-BN-TR"
 			(at 68.58 76.2 0)
 			(effects
@@
 			)
 		)
-		(property "Footprint" "Oscillator:Oscillator_DIP-14"
+		(property "Footprint" "m68030-sbc:Oscillator_SMD_ECS-3951M_7.0x5.0mm_DIP14PinMap"
 			(at 264.16 101.6 0)
 			(effects
@@
 			)
 		)
-		(property "MPN" "optional 5 V CMOS oscillator for a slower 68882"
+		(property "MPN" "ECS-3951M-200-BN-TR [VERIFY freq vs 68882 grade]"
 			(at 264.16 101.6 0)
 			(effects
@@
 			)
 		)
-		(property "Footprint" "Oscillator:Oscillator_DIP-14"
+		(property "Footprint" "m68030-sbc:Oscillator_SMD_ECS-3951M_7.0x5.0mm_DIP14PinMap"
 			(at 68.58 165.1 0)
 			(effects
@@
 			)
 		)
-		(property "MPN" "50.000 MHz 5 V CMOS oscillator"
+		(property "MPN" "ECS-3951M-500-BN-TR"
 			(at 68.58 165.1 0)
 			(effects

Commit message: PCB: fully route the 4-layer board, then fix DRAM termination, strobe stubs and clocks
Route all 499 signal connections on the 220x175 mm 4-layer board, with signals
on F.Cu/B.Cu and solid In1 GND / In2 +5V (+3V3 island). The scripted grid router
is in kicad/tools/route/ (0.4233 mm grid aligned to U1, A* + PathFinder).
Then fix signal integrity (kicad/tools/route/sifix/): strip the signal tracks,
move the parts and reroute.

Full route (first pass):
- 100 % routed, DRC 0 errors, parity 0; 2453 vias, 56.1 m of signal track.
- 55 parts nudged <= 0.212 mm onto the grid. The DNP 74ACT257 fallback
  (U801-U803, R829-R838) is set to on_board no in dram.kicad_sch.

SI fix (this board, sha1 2221a671):
- DRAM 33R R804-R824 moved to B.Cu next to U4: pad to U4 pin is now
  1.6-6.9 mm (was 2.9-27.2 mm).
- RAS0_n/CAS3_n/WE_n: LA3 J13 pins 37-39 are now NC (debug.kicad_sch).
  TP801/806/807 moved to the SIMM-side resistors.
  RAS0_n 325/17 -> 27.5 mm/1 via, CAS3_n 232/7 -> 17.8/0, WE_n 224/5 -> 17.4/1.
  TP stubs are 0 / 13.5 / 9.7 mm.
- Clock block (U10, X1, R301-R306, decaps) moved next to U4/U3. R307/R308 moved
  to the X2/X3 outputs. U10 outputs swapped in clock.kicad_sch: pin 18 CLKB_DRAMC,
  pin 14 CLKB_CPU, pin 12 CLKB_GLUE.
  CLK_EXP 147/2 -> 56/0, CLK_GLUE 109/0 -> 22/0, CLK_CPU 75/2 -> 57/0,
  CLK_DRAMC 38 -> 62, CLK_FPU_CPU 52/2 -> 70/0, DRAM_CLK 37 -> 59/0,
  X2-OUT 31/2 -> 4/0. Every CLKB_* is 1.7 mm. Clocks are ~100 % on F.Cu over GND.
  Tradeoff: CLK_LA 28 -> 202 mm/2 vias, CLKB_X3 (DNP) 51 -> 80 mm.
- Board total: 2365 vias, 53.8 m of signal track. 100 % routed, DRC 0 errors,
  0 unconnected, parity 0, ERC 0/0. 4 silk warnings (was 5). .kicad_pro unchanged.
- Note: build.py / sheet_*.py do not contain the J13 NC or the U10 swap.
- Renders: renders/m68030-sbc-routed-*.png, renders/m68030-sbc-sifix-*.png.
Connections:
- net CLKB_CPU: now also U10.14 (1Y2); no longer U10.18 (1Y0)
- net CLKB_DRAMC: now also U10.18 (1Y0); no longer U10.12 (1Y3)
- net CLKB_GLUE: now also U10.12 (1Y3); no longer U10.14 (1Y2)
Changed lines of the file:
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@@
 		)
 	)
-	(label "CLKB_CPU"
+	(label "CLKB_DRAMC"
 		(at 129.54 76.2 0)
 		(effects
@@
 		)
 	)
-	(label "CLKB_GLUE"
+	(label "CLKB_CPU"
 		(at 129.54 81.28 0)
 		(effects
@@
 		)
 	)
-	(label "CLKB_DRAMC"
+	(label "CLKB_GLUE"
 		(at 129.54 83.82 0)
 		(effects
