File: 68030-design/kicad/debug.kicad_sch (KiCad schematic)
At the start: 5 parts, among them J11 LA1 A31-A0, J12 LA2 D31-D0, J13 LA3 control

Commit message: PCB: fully route the 4-layer board, then fix DRAM termination, strobe stubs and clocks
Route all 499 signal connections on the 220x175 mm 4-layer board, with signals
on F.Cu/B.Cu and solid In1 GND / In2 +5V (+3V3 island). The scripted grid router
is in kicad/tools/route/ (0.4233 mm grid aligned to U1, A* + PathFinder).
Then fix signal integrity (kicad/tools/route/sifix/): strip the signal tracks,
move the parts and reroute.

Full route (first pass):
- 100 % routed, DRC 0 errors, parity 0; 2453 vias, 56.1 m of signal track.
- 55 parts nudged <= 0.212 mm onto the grid. The DNP 74ACT257 fallback
  (U801-U803, R829-R838) is set to on_board no in dram.kicad_sch.

SI fix (this board, sha1 2221a671):
- DRAM 33R R804-R824 moved to B.Cu next to U4: pad to U4 pin is now
  1.6-6.9 mm (was 2.9-27.2 mm).
- RAS0_n/CAS3_n/WE_n: LA3 J13 pins 37-39 are now NC (debug.kicad_sch).
  TP801/806/807 moved to the SIMM-side resistors.
  RAS0_n 325/17 -> 27.5 mm/1 via, CAS3_n 232/7 -> 17.8/0, WE_n 224/5 -> 17.4/1.
  TP stubs are 0 / 13.5 / 9.7 mm.
- Clock block (U10, X1, R301-R306, decaps) moved next to U4/U3. R307/R308 moved
  to the X2/X3 outputs. U10 outputs swapped in clock.kicad_sch: pin 18 CLKB_DRAMC,
  pin 14 CLKB_CPU, pin 12 CLKB_GLUE.
  CLK_EXP 147/2 -> 56/0, CLK_GLUE 109/0 -> 22/0, CLK_CPU 75/2 -> 57/0,
  CLK_DRAMC 38 -> 62, CLK_FPU_CPU 52/2 -> 70/0, DRAM_CLK 37 -> 59/0,
  X2-OUT 31/2 -> 4/0. Every CLKB_* is 1.7 mm. Clocks are ~100 % on F.Cu over GND.
  Tradeoff: CLK_LA 28 -> 202 mm/2 vias, CLKB_X3 (DNP) 51 -> 80 mm.
- Board total: 2365 vias, 53.8 m of signal track. 100 % routed, DRC 0 errors,
  0 unconnected, parity 0, ERC 0/0. 4 silk warnings (was 5). .kicad_pro unchanged.
- Note: build.py / sheet_*.py do not contain the J13 NC or the U10 swap.
- Renders: renders/m68030-sbc-routed-*.png, renders/m68030-sbc-sifix-*.png.
Connections:
- net CAS3_n: no longer J13.38 (Pin_38)
- net RAS0_n: no longer J13.37 (Pin_37)
- net WE_n: no longer J13.39 (Pin_39)
- no-connect marks 0 -> 3
Changed lines of the file:
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@@
 		)
 	)
+	(no_connect
+		(at 425.45 182.88)
+	)
+	(no_connect
+		(at 438.15 182.88)
+	)
+	(no_connect
+		(at 425.45 185.42)
+	)
 	(wire
 		(pts
@@
 	(wire
 		(pts
-			(xy 425.45 182.88)
-			(xy 417.83 182.88)
-		)
-		(stroke
-			(width 0)
-			(type default)
-		)
-	)
-	(wire
-		(pts
-			(xy 438.15 182.88)
-			(xy 445.77 182.88)
-		)
-		(stroke
-			(width 0)
-			(type default)
-		)
-	)
-	(wire
-		(pts
-			(xy 425.45 185.42)
-			(xy 417.83 185.42)
-		)
-		(stroke
-			(width 0)
-			(type default)
-		)
-	)
-	(wire
-		(pts
 			(xy 425.45 142.24)
 			(xy 420.37 142.24)
@@
 		)
 	)
-	(label "RAS0_n"
-		(at 417.83 182.88 180)
-		(effects
-			(font
-				(size 1.27 1.27)
-			)
-			(justify right bottom)
-		)
-	)
-	(label "CAS3_n"
-		(at 445.77 182.88 0)
-		(effects
-			(font
-				(size 1.27 1.27)
-			)
-			(justify left bottom)
-		)
-	)
-	(label "WE_n"
-		(at 417.83 185.42 180)
-		(effects
-			(font
-				(size 1.27 1.27)
-			)
-			(justify right bottom)
-		)
-	)
 	(hierarchical_label "A[0..31]"
 		(shape input)
@@
 		)
 	)
-	(text "Logic analyzer (spec §8.4). Keep the headers within about 25 mm of the CPU [EST] so the stubs stay short.\nPin order on each header: signals on every pin that is not a multiple of 5; pins 5/10/15/20/25/30/35/40 are GND.\nLA1 is A31 down to A0. LA2 is D31 down to D0. LA3 is the §8.4 list, in that order, starting at pin 1.\nLED_n and HALT_LED_n are TP1101/TP1102 only. The LEDs themselves are D701/D702 on the glue sheet."
+	(text "Logic analyzer (spec §8.4). Keep the headers within about 25 mm of the CPU [EST] so the stubs stay short.\nPin order on each header: signals on every pin that is not a multiple of 5; pins 5/10/15/20/25/30/35/40 are GND.\nLA1 is A31 down to A0. LA2 is D31 down to D0. LA3 is the §8.4 list, in that order, starting at pin 1.\nLED_n and HALT_LED_n are TP1101/TP1102 only. The LEDs themselves are D701/D702 on the glue sheet.\nSI fix 2026-10-18: LA3 pins 37/38/39 (RAS0_n/CAS3_n/WE_n) are no-connect, so the DRAM strobes have no long stub.\nProbe them at TP801/TP806/TP807, next to the SIMM-side 33R resistors."
 		(exclude_from_sim no)
 		(at 29.845 360.045 0)
