File: 68030-design/kicad/dram.kicad_sch (KiCad schematic)
At the start: 77 parts, among them J1 SIMM-72 socket, J5 JTAG U4 (ATDH1150USB), U4 ATF1508AS-7JX84, U801 74ACT257, U802 74ACT257, U803 74ACT257

Commit message: CPLD: Rev A.2 pin swap for U3 glue and U4 DRAM to match the 220x175 placement
Re-assign the U3/U4 user I/O pins to follow the bus order at the CPU, FPU,
SIMM, LA headers and DIN. Dedicated inputs, JTAG, power, jumpered pins, TP pins
and the reserved SPI pins (46/48/49) did not move.

- U3 glue: 57 pins moved; airwire length 2784 -> 2369 mm, crossings 254 -> 0.
- U4 DRAM: 54 pins moved; 1598 -> 1296 mm, crossings 372 -> 8. The search
  kept fit1508 in the loop, so all 9 cascades and the 14.0 ns timing were kept.
- Refits (fit1508 v1918, -7, JTAG on): glue 121/128 MC, 20.3 ns; DRAM 78/128 MC,
  14.0 ns (same as Rev A.1). All CPLD and system sims: 0 errors, 0 DSACK contention.
- Schematics: label edits in place in glue_cpld/dram.kicad_sch (not build.py).
  ERC 0 errors / 0 warnings.
- PCB: 111 U3/U4 pad nets updated; R804-R824 moved to B.Cu in SIMM pin order.
  DRC 0 errors, parity 0 (board still unrouted at this commit).
- FreeRouting re-test (scratch): 4L completion 27 % -> 32.5 %, 6L 25 % -> 29.9 %.
- New tools: kicad/tools/cpld_pinswap_*.py. Pin tables in cpld/*/README.md.
- .kicad_pro unchanged.
Connections:
- net A0: now also U4.34 (I/O); no longer U4.46 (I/O)
- net A1: now also U4.37 (I/O); no longer U4.45 (I/O/PD2)
- net A10: now also U4.54 (I/O); no longer U4.33 (I/O)
- net A11: now also U4.51 (I/O); no longer U4.74 (I/O)
- net A12: now also U4.65 (I/O); no longer U4.73 (I/O)
- net A13: now also U4.55 (I/O); no longer U4.70 (I/O)
- net A15: now also U4.67 (I/O); no longer U4.68 (I/O)
- net A16: now also U4.73 (I/O); no longer U4.67 (I/O)
- net A17: now also U4.52 (I/O); no longer U4.65 (I/O)
- net A18: now also U4.48 (I/O); no longer U4.64 (I/O)
- net A19: now also U4.49 (I/O); no longer U4.63 (I/O)
- net A2: now also U4.60 (I/O); no longer U4.44 (I/O)
- net A20: now also U4.80 (I/O); no longer U4.61 (I/O)
- net A21: now also U4.45 (I/O/PD2); no longer U4.60 (I/O)
- net A22: now also U4.46 (I/O); no longer U4.58 (I/O)
- net A23: now also U4.44 (I/O); no longer U4.57 (I/O)
- net A24: now also U4.41 (I/O); no longer U4.56 (I/O)
- net A25: now also U4.40 (I/O); no longer U4.55 (I/O)
- net A26: now also U4.39 (I/O); no longer U4.54 (I/O)
- net A3: now also U4.64 (I/O); no longer U4.41 (I/O)
- net A4: now also U4.58 (I/O); no longer U4.40 (I/O)
- net A5: now also U4.68 (I/O); no longer U4.39 (I/O)
- net A6: now also U4.61 (I/O); no longer U4.37 (I/O)
- net A7: now also U4.56 (I/O); no longer U4.36 (I/O)
- net A8: now also U4.57 (I/O); no longer U4.35 (I/O)
- net A9: now also U4.63 (I/O); no longer U4.34 (I/O)
- net DRAM_SEL_n: now also U4.33 (I/O); no longer U4.52 (I/O)
- net DSACK0_n: now also U4.28 (I/O); no longer U4.12 (I/O/PD1)
- net DSACK1_n: now also U4.30 (I/O); no longer U4.15 (I/O)
- net MUX_SEL: now also U4.74 (I/O); no longer U4.80 (I/O)
- net R_W: now also U4.31 (I/O); no longer U4.51 (I/O)
- net SIZ0: now also U4.36 (I/O); no longer U4.49 (I/O)
- net SIZ1: now also U4.35 (I/O); no longer U4.48 (I/O)
- net U4_CAS0_n: now also U4.4 (I/O); no longer U4.11 (I/O)
- net U4_CAS1_n: now also U4.77 (I/O); no longer U4.75 (I/O)
- net U4_CAS2_n: now also U4.70 (I/O); no longer U4.76 (I/O)
- net U4_CAS3_n: now also U4.79 (I/O); no longer U4.77 (I/O)
- net U4_MA0: now also U4.22 (I/O); no longer U4.20 (I/O)
- net U4_MA1: now also U4.20 (I/O); no longer U4.21 (I/O)
- net U4_MA10: now also U4.10 (I/O); no longer U4.4 (I/O)
- net U4_MA11: now also U4.9 (I/O); no longer U4.5 (I/O)
- net U4_MA2: now also U4.25 (I/O); no longer U4.22 (I/O)
- net U4_MA3: now also U4.21 (I/O); no longer U4.24 (I/O)
- net U4_MA4: now also U4.24 (I/O); no longer U4.25 (I/O)
- net U4_MA5: now also U4.15 (I/O); no longer U4.27 (I/O)
- net U4_MA6: now also U4.12 (I/O/PD1); no longer U4.28 (I/O)
- net U4_MA7: now also U4.11 (I/O); no longer U4.29 (I/O)
- net U4_MA8: now also U4.27 (I/O); no longer U4.30 (I/O)
- net U4_MA9: now also U4.29 (I/O); no longer U4.31 (I/O)
- net U4_RAS0_n: now also U4.76 (I/O); no longer U4.6 (I/O)
- net U4_RAS1_n: now also U4.5 (I/O); no longer U4.8 (I/O)
- net U4_RAS2_n: now also U4.6 (I/O); no longer U4.9 (I/O)
- net U4_RAS3_n: now also U4.8 (I/O); no longer U4.10 (I/O)
- net U4_WE_n: now also U4.75 (I/O); no longer U4.79 (I/O)
Other:
- note added: "FITTED PINOUT: Yosys + hoglet67/atf15xx_yosys -> Microchip fit1508.exe v1918 (Wine), ATF1508AS PLCC84 -7, JTAG ON, pins locked (-preassign keep), -optimize on, -pin_keep on. Result: 80/128 macrocells, 52 flip-flops, 210 product terms; 55/60 user I/O + 4 JTAG + 3/4 dedicated inputs. Worst register-to-register 14.0 ns (50 MHz = 20 ns met). Rev A.2 (2026-10-17): I/O pins re-assigned for the 220x175 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"
- note added: "Not needed: U4 fits with the MA mux inside (80/128 MC, 50 MHz met). To use: fit U801-U803 + C818-C820 and R829-R838, remove R806-R815 (U4 MA2-MA11 path), and rebuild dram.v with MA2-MA11 unused. S = MUX_SEL (U4 pin 74; low = row on I0, high = column on I1). 74ACT257 tpd <= 10.5 ns (onsemi MC74ACT257), vs 7.5-10 ns in U4."
- note removed: "FITTED PINOUT: Yosys + hoglet67/atf15xx_yosys -> Microchip fit1508.exe v1918 (Wine), ATF1508AS PLCC84 -7, JTAG ON, pins locked (-preassign keep), -optimize on, -pin_keep on. Result: 80/128 macrocells, 52 flip-flops, 210 product terms; 55/60 user I/O + 4 JTAG + 3/4 dedicated inputs. Worst register-to-register 14.0 ns (50 MHz = 20 ns met). Sources, reports, JEDEC, testbench: cpld/dram/ (dram.v, dra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"
- note removed: "Not needed: U4 fits with the MA mux inside (80/128 MC, 50 MHz met). To use: fit U801-U803 + C818-C820 and R829-R838, remove R806-R815 (U4 MA2-MA11 path), and rebuild dram.v with MA2-MA11 unused. S = MUX_SEL (U4 pin 80; low = row on I0, high = column on I1). 74ACT257 tpd <= 10.5 ns (onsemi MC74ACT257), vs 7.5-10 ns in U4."
